Commit message: integracion de gazebo

File: src/robot_description/urdf/robot_description.urdf (robot description, URDF)
Before this commit: robot robot_description, 54 links, 53 joints
Joints:
- joint Motorreductor_37D_con_encoder_1__CLM_Llanta60mmD_2: axis 1 0 0 -> -1 0 0
- joint Motorreductor_37D_con_encoder_2__CLM_Llanta60mmD_1: axis 1 0 0 -> -1 0 0
